File: Cyberdeck/IOConfig.kicad_sch (KiCad schematic)
At the start: 14 parts, among them SW10 Push Button, SW4 Push Button, SW5 Push Button, SW6 Push Button, SW7 Push Button, SW8 Push Button, SW9 Push Button

Commit message: Finished schematic
Parts:
- added H2: 16pin Header, lcsc_footprints:C2894939_HDR-TH_16P-P2_54-V-M, symbol lcsc_imported:PZ254-1-16-Z-8_5
- renumbered R14 to R17, R15 to R18, R16 to R19, R17 to R20, R18 to R21, R19 to R22, R20 to R23, SW9 to SW10, SW10 to SW11, SW4 to SW5, SW5 to SW6, SW6 to SW7, SW7 to SW8, SW8 to SW9
Connections:
- net GND: now also H2.1
- net PB3: now also H2.4; no longer R17.2, SW5.1
- net PB4: now also H2.5; no longer R18.2, SW6.1
- net PB5: now also H2.6; no longer R19.2, SW7.1
- net PB6: now also H2.7; no longer R20.2, SW8.1
- net PB7: now also H2.9; no longer R21.2, SW9.1
- net PB8: now also H2.10; no longer R22.2, SW10.1
- net PB9: now also H2.11; no longer R23.2, SW11.1
- net Vdd renamed V_IN
- net V_IN: now also H2.2
- new net Backlight: H2.8
- new net PA2: R17.2, SW5.1
- new net PA3: R18.2, SW6.1
- new net PA4: R19.2, SW7.1
- new net PA5: R20.2, SW8.1
- new net PA6: R21.2, SW9.1
- new net PA7: R22.2, SW10.1
- new net PA8: R23.2, SW11.1
- new net PB1: H2.3
- new net PB10: H2.12
- new net PB12: H2.13
- new net PB13: H2.14
- new net PB14: H2.15
- new net PB15: H2.16
Other:
- note added: "These are the inputs to the ILI9341 3.2" TFT display screen for 8bit mode"
- moved on the sheet: R17, R18, R19, R20, R21, R22, R23, SW10, SW11, SW5, SW6, SW7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

Commit message: Rerouted vias, optimized layout, and added pwr/gnd planes
Connections:
- net V_IN renamed V_REG
Changed lines of the file:
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@@
 		)
 	)
-	(hierarchical_label "V_IN"
+	(hierarchical_label "V_REG"
 		(shape input)
 		(at 205.74 43.18 90)
