File: Cyberdeck/MicroController.kicad_sch (KiCad schematic)
At the start: 26 parts, among them SW1 Push Button, SW2 Push Button, SW3 Push Button, U3 STM32F411CEU6, X1 32.768KHz 12.5pF, X2 25MHZ 12PF 10PPM

Commit message: Finished schematic
Parts:
- added LED3: 2.3v Red, lcsc_footprints:C965799_LED0603-RD_RED, symbol lcsc_imported:XL-1608SURC-06
- added R12: 100Ω, lcsc_footprints:C2906981_R0603, symbol lcsc_imported:FRC0603F1000TS
- renumbered C14 to C10, C9 to C11, C11 to C12, C10 to C13, C17 to C14, C13 to C15, C12 to C16, C19 to C17, C16 to C8, C15 to C9, R22 to R13, R12 to R14, R13 to R15, R21 to R16, SW1 to SW2, SW2 to SW3, SW3 to SW4, U3 to U5
Connections:
- net V_OUT is gone; now on net V_IN: C10.1, C13.2, C14.1, C7.2, C8.1, C9.1, H1.1, SW2.2, SW3.2, U5.1 (VBAT), U5.24 (VDD), U5.36 (VDD), U5.48 (VDD), U5.9 (VDDA/VREF+)
- net GND: now also LED3.1 (K)
- net PA1 renamed LED
- net LED: now also R12.2
- new net: LED3.2 (A), R12.1
Other:
- moved on the sheet: R10, SW2

Commit message: Rerouted vias, optimized layout, and added pwr/gnd planes
Connections:
- net V_IN renamed V_REG
- net V_REG: no longer R13.1, USB1.A4B9 (VBUS), USB1.B4A9 (VBUS)
- new net V_USB: R13.1, USB1.A4B9 (VBUS), USB1.B4A9 (VBUS)
Changed lines of the file:
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@@
 		)
 	)
-	(hierarchical_label "V_OUT"
+	(hierarchical_label "V_USB"
 		(shape output)
 		(at 135.89 143.51 0)
@@
 		)
 	)
-	(hierarchical_label "V_IN"
+	(hierarchical_label "V_REG"
 		(shape input)
 		(at 195.58 19.05 0)

Commit message: Finalized PCB; Made gerber files
Parts:
- removed C10, C14, C17, C8, C9: 100nF, lcsc_footprints:C1591_C0603, symbol lcsc_imported:100nF_(104)_±10%_50V
- added C10, C14, C17, C8, C9: 100nF, lcsc_footprints:C66501_C0603, symbol lcsc_imported:CL10B104KO8NNNC
- added D1, D2: ESD321, lcsc_footprints:C2868952_X1SON-2_L1_0-W0_6-P0_65-RD-1, symbol lcsc_imported:ESD321DPYR_C2868952
- added D3: ESDA7P60, lcsc_footprints:C1975146_D1610-RD, symbol lcsc_imported:ESDA7P60-1U1M
- renumbered R14 to R13, R15 to R14, R13 to R15
Connections:
- net DN: now also D2.1 (I/O)
- net DP: now also D1.1 (I/O)
- net GND: now also C10.1, C14.1, C17.1, C8.1, C9.1, D1.2 (GND), D2.2 (GND), D3.2 (A)
- net NRST: now also C17.2
- net V_REG: now also C10.2, C14.2, C8.2, C9.2
- net V_USB: now also D3.1 (C)
Other:
- moved on the sheet: R13, R14, R15, R16
